File: Matchstick 3.0.kicad_pcb (KiCad board)
At the start: 2 copper layers, 47.2 x 34 mm, 11 parts, among them J3 Barrel_Jack, J4 Screw_Terminal_01x08, SW1 SparkFun_COM-08720, U1 M5StampS3

Commit message: sent to jlcpcb
Other:
- board text added: "JLCJLCJLCJLC"
- board text removed: "WayWayWay"
Changed lines of the file:
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@@
 	)
 	(paper "A4")
+	(title_block
+		(title "Matchstick 3.0 (Barrel Jack)")
+		(date "2026-01-26")
+		(company "0x76656E Labs")
+	)
 	(layers
 		(0 "F.Cu" signal)
@@
 		)
 		(pad_to_mask_clearance 0)
-		(solder_mask_min_width 0.1016)
 		(allow_soldermask_bridges_in_footprints no)
 		(tenting front back)
@@
 		)
 	)
-	(gr_text "WayWayWay"
+	(gr_text "JLCJLCJLCJLC"
 		(at 192 118.95 0)
 		(layer "B.SilkS")
